File: cad/kicad/project/pcb.kicad_sch (KiCad schematic)
At the start: 6 parts, among them J1 USB_A, J2 USB_C_Receptacle_USB2.0, U4 PiPico

Commit message: Updated Freecad data
Parts:
- J1: footprint custom_lib:USB A Port -> somnos_lib:USB A Port
- J2: footprint custom_lib:USB C Port -> somnos_lib:USB C Port
- U1: footprint custom_lib:END28J60 -> somnos_lib:END28J60; symbol custom_lib:ENC28J60 -> somnos_lib:ENC28J60
- U2: footprint custom_lib:INA219 -> somnos_lib:INA219; symbol custom_lib:INA219 -> somnos_lib:INA219
- U3: footprint custom_lib:N-MOS_1 -> somnos_lib:N-MOS_1; symbol custom_lib:N-MOS_x2_module -> somnos_lib:N-MOS_x2_module
- U4: footprint custom_lib:PiPico -> somnos_lib:PiPico; symbol custom_lib:PiPico -> somnos_lib:PiPico
Changed lines of the file:
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@@
     (effects (font (size 1.27 1.27)) (justify left bottom))
   )
-  (symbol (lib_id "custom_lib:N-MOS_x2_module") (at 107.95 54.61 0) (unit 1)
+  (symbol (lib_id "somnos_lib:N-MOS_x2_module") (at 107.95 54.61 0) (unit 1)
     (in_bom yes) (on_board yes) (dnp no) (fields_autoplaced)
     (property "Reference" "U3" (at 107.315 43.18 0)
@@
       (effects (font (size 1.27 1.27)))
     )
-    (property "Footprint" "custom_lib:N-MOS_1" (at 111.76 66.04 0)
+    (property "Footprint" "somnos_lib:N-MOS_1" (at 111.76 66.04 0)
       (effects (font (size 1.27 1.27)) hide)
     )
@@
     )
   )
-  (symbol (lib_id "custom_lib:ENC28J60") (at 49.53 144.78 180) (unit 1)
+  (symbol (lib_id "somnos_lib:ENC28J60") (at 49.53 144.78 180) (unit 1)
     (in_bom yes) (on_board yes) (dnp no) (fields_autoplaced)
     (property "Reference" "U1" (at 49.53 129.54 0)
@@
       (effects (font (size 1.27 1.27)))
     )
-    (property "Footprint" "custom_lib:END28J60" (at 49.53 144.78 0)
+    (property "Footprint" "somnos_lib:END28J60" (at 49.53 144.78 0)
       (effects (font (size 1.27 1.27)) hide)
     )
@@
     )
   )
-  (symbol (lib_id "custom_lib:INA219") (at 170.18 53.34 0) (unit 1)
+  (symbol (lib_id "somnos_lib:INA219") (at 170.18 53.34 0) (unit 1)
     (in_bom yes) (on_board yes) (dnp no) (fields_autoplaced)
     (property "Reference" "U2" (at 169.545 41.91 0)
@@
       (effects (font (size 1.27 1.27)))
     )
-    (property "Footprint" "custom_lib:INA219" (at 170.18 53.34 0)
+    (property "Footprint" "somnos_lib:INA219" (at 170.18 53.34 0)
       (effects (font (size 1.27 1.27)) hide)
     )
@@
       (effects (font (size 1.27 1.27)))
     )
-    (property "Footprint" "custom_lib:USB A Port" (at 36.83 59.69 0)
+    (property "Footprint" "somnos_lib:USB A Port" (at 36.83 59.69 0)
       (effects (font (size 1.27 1.27)) hide)
     )
@@
     )
   )
-  (symbol (lib_id "custom_lib:PiPico") (at 101.6 134.62 0) (unit 1)
+  (symbol (lib_id "somnos_lib:PiPico") (at 101.6 134.62 0) (unit 1)
     (in_bom yes) (on_board yes) (dnp no) (fields_autoplaced)
     (property "Reference" "U4" (at 101.6 95.25 0)
@@
       (effects (font (size 1.27 1.27)))
     )
-    (property "Footprint" "custom_lib:PiPico" (at 101.6 134.62 0)
+    (property "Footprint" "somnos_lib:PiPico" (at 101.6 134.62 0)
       (effects (font (size 1.27 1.27)) hide)
     )
@@
       (effects (font (size 1.27 1.27)) (justify right))
     )
-    (property "Footprint" "custom_lib:USB C Port" (at 217.17 63.5 0)
+    (property "Footprint" "somnos_lib:USB C Port" (at 217.17 63.5 0)
       (effects (font (size 1.27 1.27)) hide)
     )
